File: Power Monitor.kicad_sch (KiCad schematic)
At the start: 7 parts, among them J12 Conn_01x02, U9 INA219BIDR

Commit message: Set PCB metadata
Other:
- title: (none) -> BenchATX Power Monitor
Changed lines of the file:
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@@
 (kicad_sch (version 20230121) (generator eeschema)
   (paper "A4")
+  (title_block
+    (title "BenchATX Power Monitor")
+    (date "2026-05-01")
+    (rev "A")
+  )
   (junction (at 74.93 46.99) (diameter 0) (color 0 0 0 0)
   )
